Commit message: Making the Crab Body

File: body1.urdf (robot description, URDF)
Before this commit: robot robot, 19 links, 18 joints
Links:
- removed link FrontLeftArm
- removed link FrontLeftClaw
- removed link FrontLeftClawTip
- removed link FrontRightArm
- removed link FrontRightClaw
- removed link FrontRightClawTip
- link Torso: mass 10.0 -> 1.0; geometry collision box size=2 1 1; visual box size=2 1 1
Joints:
- removed joint FrontLeftArm_FrontLeftClaw
- removed joint FrontLeftClaw_FrontLeftClawTip
- removed joint FrontRightArm_FrontRightClaw
- removed joint FrontRightClaw_FrontRightClawTip
- removed joint Torso_FrontLeftArm
- removed joint Torso_FrontRightArm
- joint Torso_BackLeftLeg: origin xyz=-0.5 -0.5 1.0 rpy=0 0 0 -> xyz=-0.5 -0.25 1.0 rpy=0 0 0
- joint Torso_BackRightLeg: origin xyz=0.5 -0.5 1.0 rpy=0 0 0 -> xyz=0.5 -0.25 1.0 rpy=0 0 0
- joint Torso_FrontLeftLeg: origin xyz=-0.5 0.5 1.0 rpy=0 0 0 -> xyz=-0.5 0.25 1.0 rpy=0 0 0
- joint Torso_FrontRightLeg: origin xyz=0.5 0.5 1.0 rpy=0 0 0 -> xyz=0.5 0.25 1.0 rpy=0 0 0

Commit message: finish Mr Krabs

File: body1.urdf (robot description, URDF)
Before this commit: robot robot, 19 links, 18 joints
Joints:
- joint Torso_BackLeftLeg: axis 0 1 0 -> 0 0 1
- joint Torso_BackRightLeg: axis 0 1 0 -> 0 0 1
- joint Torso_FrontLeftLeg: axis 0 1 0 -> 0 0 1
- joint Torso_FrontRightLeg: axis 0 1 0 -> 0 0 1
- joint Torso_MiddleLeftLeg: axis 0 1 0 -> 0 0 1
- joint Torso_MiddleRightLeg: axis 0 1 0 -> 0 0 1
