Commit message: finish E

File: body.urdf (robot description, URDF)
Before this commit: robot robot, 3 links, 2 joints
Joints:
- removed joint Link1_Link2
- added joint Link0_Link2: type revolute, parent Link0, child Link2, origin xyz=2.0 0 1.0 rpy=0 0 0, axis 0 1 0, limit lower=-3.14159 upper=3.14159 effort=0.0 velocity=0.0
- joint Link0_Link1: origin xyz=0.5 0 1.0 rpy=0 0 0 -> xyz=1.0 0 1.0 rpy=0 0 0

Commit message: rename variables and add back leg sensor to simulate

File: body.urdf (robot description, URDF)
Before this commit: robot robot, 3 links, 2 joints
Links:
- removed link Link0
- removed link Link1
- removed link Link2
- added link BackLeg, mass 1; collision box size=1 1 1; visual box size=1 1 1
- added link FrontLeg, mass 1; collision box size=1 1 1; visual box size=1 1 1
- added link Torso, mass 1; collision box size=1 1 1; visual box size=1 1 1
Joints:
- removed joint Link0_Link1
- removed joint Link0_Link2
- added joint Torso_BackLeg: type revolute, parent Torso, child BackLeg, origin xyz=1.0 0 1.0 rpy=0 0 0, axis 0 1 0, limit lower=-3.14159 upper=3.14159 effort=0.0 velocity=0.0
- added joint Torso_FrontLeg: type revolute, parent Torso, child FrontLeg, origin xyz=2.0 0 1.0 rpy=0 0 0, axis 0 1 0, limit lower=-3.14159 upper=3.14159 effort=0.0 velocity=0.0

Commit message: finish front leg

File: body.urdf (robot description, URDF)
Before this commit: robot robot, 3 links, 2 joints
Links:
- link FrontLeg: geometry collision box size=0.2 1 0.2; visual box size=0.2 1 0.2
Joints:
- joint Torso_BackLeg: origin xyz=1.0 0 1.0 rpy=0 0 0 -> xyz=10.0 0 1.0 rpy=0 0 0
- joint Torso_FrontLeg: origin xyz=2.0 0 1.0 rpy=0 0 0 -> xyz=0 0.5 1.0 rpy=0 0 0

Commit message: finish changing joint axes

File: body.urdf (robot description, URDF)
Before this commit: robot robot, 3 links, 2 joints
Links:
- link BackLeg: geometry collision box size=0.2 1 0.2; visual box size=0.2 1 0.2
Joints:
- joint Torso_BackLeg: axis 0 1 0 -> 1 0 0; origin xyz=10.0 0 1.0 rpy=0 0 0 -> xyz=0 -0.5 1.0 rpy=0 0 0
- joint Torso_FrontLeg: axis 0 1 0 -> 1 0 0

Commit message: finish left and right legs

File: body.urdf (robot description, URDF)
Before this commit: robot robot, 3 links, 2 joints
Links:
- added link LeftLeg, mass 1; collision box size=1 0.2 0.2; visual box size=1 0.2 0.2
- added link RightLeg, mass 1; collision box size=1 0.2 0.2; visual box size=1 0.2 0.2
Joints:
- added joint Torso_LeftLeg: type revolute, parent Torso, child LeftLeg, origin xyz=-0.5 0 1.0 rpy=0 0 0, axis 0 1 0, limit lower=-3.14159 upper=3.14159 effort=0.0 velocity=0.0
- added joint Torso_RightLeg: type revolute, parent Torso, child RightLeg, origin xyz=0.5 0 1.0 rpy=0 0 0, axis 0 1 0, limit lower=-3.14159 upper=3.14159 effort=0.0 velocity=0.0

Commit message: finish creating robot body and brain

File: body.urdf (robot description, URDF)
Before this commit: robot robot, 5 links, 4 joints
Links:
- added link LowerBackLeg, mass 1; collision box size=0.2 0.2 1; visual box size=0.2 0.2 1
- added link LowerFrontLeg, mass 1; collision box size=0.2 0.2 1; visual box size=0.2 0.2 1
- added link LowerLeftLeg, mass 1; collision box size=0.2 0.2 1; visual box size=0.2 0.2 1
- added link LowerRightLeg, mass 1; collision box size=0.2 0.2 1; visual box size=0.2 0.2 1
Joints:
- added joint BackLeg_LowerBackLeg: type revolute, parent BackLeg, child LowerBackLeg, origin xyz=0 -1 0 rpy=0 0 0, axis 1 0 0, limit lower=-3.14159 upper=3.14159 effort=0.0 velocity=0.0
- added joint FrontLeg_LowerFrontLeg: type revolute, parent FrontLeg, child LowerFrontLeg, origin xyz=0 1 0 rpy=0 0 0, axis 1 0 0, limit lower=-3.14159 upper=3.14159 effort=0.0 velocity=0.0
- added joint LeftLeg_LowerLeftLeg: type revolute, parent LeftLeg, child LowerLeftLeg, origin xyz=-1 0 0 rpy=0 0 0, axis 0 1 0, limit lower=-3.14159 upper=3.14159 effort=0.0 velocity=0.0
- added joint RightLeg_LowerRightLeg: type revolute, parent RightLeg, child LowerRightLeg, origin xyz=1 0 0 rpy=0 0 0, axis 0 1 0, limit lower=-3.14159 upper=3.14159 effort=0.0 velocity=0.0

Commit message: fixed mass assignments

File: body.urdf (robot description, URDF)
Before this commit: robot robot, 9 links, 8 joints
Links:
- link BackLeg: mass 1 -> 1.0
- link FrontLeg: mass 1 -> 1.0
- link LeftLeg: mass 1 -> 1.0
- link LowerBackLeg: mass 1 -> 1.0
- link LowerFrontLeg: mass 1 -> 1.0
- link LowerLeftLeg: mass 1 -> 1.0
- link LowerRightLeg: mass 1 -> 1.0
- link RightLeg: mass 1 -> 1.0
- link Torso: mass 1 -> 1.0

Commit message: Ready to run long optimization

File: body.urdf (robot description, URDF)
Before this commit: robot robot, 19 links, 18 joints
Links:
- link FrontLeftClawTip: geometry collision box size=0.1 0.4 0.1; visual box size=0.1 0.4 0.1
- link FrontRightClawTip: geometry collision box size=0.1 0.4 0.1; visual box size=0.1 0.4 0.1
- link Torso: geometry collision box size=1 1.5 1; visual mesh filename=Crab18.obj scale=5 5 5

File: body1.urdf (robot description, URDF)
Before this commit: robot robot, 13 links, 12 joints
Links:
- added link FrontLeftArm, mass 0.5; collision box size=0.2 1 0.2; visual box size=0.2 1 0.2
- added link FrontLeftClaw, mass 0.25; collision box size=0.2 0.2 1; visual box size=0.2 0.2 1
- added link FrontLeftClawTip, mass 0.25; collision box size=0.1 0.4 0.1; visual box size=0.1 0.4 0.1
- added link FrontRightArm, mass 0.5; collision box size=0.2 1 0.2; visual box size=0.2 1 0.2
- added link FrontRightClaw, mass 0.25; collision box size=0.2 0.2 1; visual box size=0.2 0.2 1
- added link FrontRightClawTip, mass 0.25; collision box size=0.1 0.4 0.1; visual box size=0.1 0.4 0.1
- link Torso: mass 1.0 -> 10.0; geometry collision box size=1 1.5 1; visual box size=1 1.5 1
Joints:
- added joint FrontLeftArm_FrontLeftClaw: type revolute, parent FrontLeftArm, child FrontLeftClaw, origin xyz=0 1 0 rpy=0 0 0, axis 0 1 0, limit lower=-3.14159 upper=3.14159 effort=0.0 velocity=0.0
- added joint FrontLeftClaw_FrontLeftClawTip: type revolute, parent FrontLeftClaw, child FrontLeftClawTip, origin xyz=0 0 1 rpy=0 0 0, axis 1 0 0, limit lower=-3.14159 upper=3.14159 effort=0.0 velocity=0.0
- added joint FrontRightArm_FrontRightClaw: type revolute, parent FrontRightArm, child FrontRightClaw, origin xyz=0 1 0 rpy=0 0 0, axis 0 1 0, limit lower=-3.14159 upper=3.14159 effort=0.0 velocity=0.0
- added joint FrontRightClaw_FrontRightClawTip: type revolute, parent FrontRightClaw, child FrontRightClawTip, origin xyz=0 0 1 rpy=0 0 0, axis 1 0 0, limit lower=-3.14159 upper=3.14159 effort=0.0 velocity=0.0
- added joint Torso_FrontLeftArm: type spherical, parent Torso, child FrontLeftArm, origin xyz=-0.25 0.5 1.25 rpy=0 0 0, axis 0 0 1, limit lower=-3.14159 upper=3.14159 effort=0.0 velocity=0.0
- added joint Torso_FrontRightArm: type revolute, parent Torso, child FrontRightArm, origin xyz=0.25 0.5 1.25 rpy=0 0 0, axis 0 0 1, limit lower=-3.14159 upper=3.14159 effort=0.0 velocity=0.0
- joint Torso_BackLeftLeg: origin xyz=-0.5 -0.25 1.0 rpy=0 0 0 -> xyz=-0.5 -0.5 1.0 rpy=0 0 0
- joint Torso_BackRightLeg: origin xyz=0.5 -0.25 1.0 rpy=0 0 0 -> xyz=0.5 -0.5 1.0 rpy=0 0 0
- joint Torso_FrontLeftLeg: origin xyz=-0.5 0.25 1.0 rpy=0 0 0 -> xyz=-0.5 0.5 1.0 rpy=0 0 0
- joint Torso_FrontRightLeg: origin xyz=0.5 0.25 1.0 rpy=0 0 0 -> xyz=0.5 0.5 1.0 rpy=0 0 0

Commit message: create body working, minus joints

File: body.urdf (robot description, URDF)
Before this commit: robot robot, 19 links, 18 joints
Links:
- removed link BackLeftLeg
- removed link BackRightLeg
- removed link FrontLeftArm
- removed link FrontLeftClaw
- removed link FrontLeftClawTip
- removed link FrontLeftLeg
- removed link FrontRightArm
- removed link FrontRightClaw
- removed link FrontRightClawTip
- removed link FrontRightLeg
- removed link LowerBackLeftLeg
- removed link LowerBackRightLeg
- removed link LowerFrontLeftLeg
- removed link LowerFrontRightLeg
- removed link LowerMiddleLeftLeg
- removed link LowerMiddleRightLeg
- removed link MiddleLeftLeg
- removed link MiddleRightLeg
- removed link Torso
- added link 0, mass 0.4011870902957314; collision box size=0.6726930718560755 0.6258901893297387 0.9528660432296472; visual box size=0.6726930718560755 0.6258901893297387 0.9528660432296472
- added link 1, mass 0.5376637462592151; collision box size=0.7077990772252228 0.8004814048813302 0.9489635118315292; visual box size=0.7077990772252228 0.8004814048813302 0.9489635118315292
- added link 10, mass 0.2376768190900014; collision box size=0.5503680142482756 0.6799789318599903 0.6350942540501034; visual box size=0.5503680142482756 0.6799789318599903 0.6350942540501034
- added link 2, mass 0.3566507896058561; collision box size=0.6774918467528679 0.5543721122675219 0.9495935189176137; visual box size=0.6774918467528679 0.5543721122675219 0.9495935189176137
- added link 3, mass 0.3857283915084767; collision box size=0.6886849246465296 0.9378505196632156 0.5972104611287365; visual box size=0.6886849246465296 0.9378505196632156 0.5972104611287365
- added link 4, mass 0.4568745767982778; collision box size=0.9802825346114531 0.5008067660526505 0.9306267661530083; visual box size=0.9802825346114531 0.5008067660526505 0.9306267661530083
- added link 5, mass 0.33098706711007536; collision box size=0.5922924746849747 0.7805479483884592 0.7159376852946082; visual box size=0.5922924746849747 0.7805479483884592 0.7159376852946082
- added link 6, mass 0.42786150274574986; collision box size=0.8483374618754722 0.8074456872650156 0.6246277111043317; visual box size=0.8483374618754722 0.8074456872650156 0.6246277111043317
- added link 7, mass 0.1998082673115593; collision box size=0.5935677419564591 0.6090741802997048 0.5526790133204857; visual box size=0.5935677419564591 0.6090741802997048 0.5526790133204857
- added link 8, mass 0.6037534067659668; collision box size=0.8177599765967094 0.8852082769781682 0.8340426837893857; visual box size=0.8177599765967094 0.8852082769781682 0.8340426837893857
- added link 9, mass 0.2376768190900014; collision box size=0.5503680142482756 0.6799789318599903 0.6350942540501034; visual box size=0.5503680142482756 0.6799789318599903 0.6350942540501034
Joints:
- removed joint BackLeftLeg_LowerBackLeftLeg
- removed joint BackRightLeg_LowerBackRightLeg
- removed joint FrontLeftArm_FrontLeftClaw
- removed joint FrontLeftClaw_FrontLeftClawTip
- removed joint FrontLeftLeg_LowerFrontLeftLeg
- removed joint FrontRightArm_FrontRightClaw
- removed joint FrontRightClaw_FrontRightClawTip
- removed joint FrontRightLeg_LowerFrontRightLeg
- removed joint MiddleLeftLeg_LowerMiddleLeftLeg
- removed joint MiddleRightLeg_LowerMiddleRightLeg
- removed joint Torso_BackLeftLeg
- removed joint Torso_BackRightLeg
- removed joint Torso_FrontLeftArm
- removed joint Torso_FrontLeftLeg
- removed joint Torso_FrontRightArm
- removed joint Torso_FrontRightLeg
- removed joint Torso_MiddleLeftLeg
- removed joint Torso_MiddleRightLeg
- added joint 0_1: type revolute, parent 0, child 1, origin xyz=0.33634653592803776 0.31294509466486936 2 rpy=0 0 0, axis 1 0 0, limit lower=-3.14159 upper=3.14159 effort=0.0 velocity=0.0
- added joint 1_2: type revolute, parent 1, child 2, origin xyz=0.7077990772252228 0.4002407024406651 0.4744817559157646 rpy=0 0 0, axis 1 0 0, limit lower=-3.14159 upper=3.14159 effort=0.0 velocity=0.0
- added joint 2_3: type revolute, parent 2, child 3, origin xyz=0.6774918467528679 0.27718605613376096 0.47479675945880684 rpy=0 0 0, axis 1 0 0, limit lower=-3.14159 upper=3.14159 effort=0.0 velocity=0.0
- added joint 3_4: type revolute, parent 3, child 4, origin xyz=0.6886849246465296 0.4689252598316078 0.2986052305643683 rpy=0 0 0, axis 1 0 0, limit lower=-3.14159 upper=3.14159 effort=0.0 velocity=0.0
- added joint 4_5: type revolute, parent 4, child 5, origin xyz=0.9802825346114531 0.25040338302632525 0.46531338307650416 rpy=0 0 0, axis 1 0 0, limit lower=-3.14159 upper=3.14159 effort=0.0 velocity=0.0
- added joint 5_6: type revolute, parent 5, child 6, origin xyz=0.5922924746849747 0.3902739741942296 0.3579688426473041 rpy=0 0 0, axis 1 0 0, limit lower=-3.14159 upper=3.14159 effort=0.0 velocity=0.0
- added joint 6_7: type revolute, parent 6, child 7, origin xyz=0.8483374618754722 0.4037228436325078 0.31231385555216584 rpy=0 0 0, axis 1 0 0, limit lower=-3.14159 upper=3.14159 effort=0.0 velocity=0.0
- added joint 7_8: type revolute, parent 7, child 8, origin xyz=0.5935677419564591 0.3045370901498524 0.2763395066602429 rpy=0 0 0, axis 1 0 0, limit lower=-3.14159 upper=3.14159 effort=0.0 velocity=0.0
- added joint 8_9: type revolute, parent 8, child 9, origin xyz=0.8177599765967094 0.4426041384890841 0.41702134189469287 rpy=0 0 0, axis 1 0 0, limit lower=-3.14159 upper=3.14159 effort=0.0 velocity=0.0
- added joint 9_10: type revolute, parent 9, child 10, origin xyz=0.5503680142482756 0.3399894659299951 0.3175471270250517 rpy=0 0 0, axis 1 0 0, limit lower=-3.14159 upper=3.14159 effort=0.0 velocity=0.0

Commit message: Get simulation to show

File: body.urdf (robot description, URDF)
Before this commit: robot robot, 11 links, 10 joints
Links:
- removed link 10
- removed link 5
- removed link 6
- removed link 7
- removed link 8
- removed link 9
- link 0: mass 0.4011870902957314 -> 0.42795200418098583; geometry collision box size=0.6836061308733558 0.8205073348040821 0.7629685700648337; visual box size=0.6836061308733558 0.8205073348040821 0.7629685700648337
- link 1: mass 0.5376637462592151 -> 0.3085508128028748; geometry collision box size=0.5657439284557486 0.6225085916630834 0.8761156600805267; visual box size=0.5657439284557486 0.6225085916630834 0.8761156600805267
- link 2: mass 0.3566507896058561 -> 0.24917680061749625; geometry collision box size=0.5837946711273645 0.5737151603948263 0.7439626840514355; visual box size=0.5837946711273645 0.5737151603948263 0.7439626840514355
- link 3: mass 0.3857283915084767 -> 0.5975508983060559; geometry collision box size=0.9694126675599994 0.8147655514340892 0.7565428907632812; visual box size=0.9694126675599994 0.8147655514340892 0.7565428907632812
- link 4: mass 0.4568745767982778 -> 0.5975508983060559; geometry collision box size=0.9694126675599994 0.8147655514340892 0.7565428907632812; visual box size=0.9694126675599994 0.8147655514340892 0.7565428907632812
Joints:
- removed joint 4_5
- removed joint 5_6
- removed joint 6_7
- removed joint 7_8
- removed joint 8_9
- removed joint 9_10
- joint 0_1: origin xyz=0.33634653592803776 0.31294509466486936 2 rpy=0 0 0 -> xyz=0.3418030654366779 0.41025366740204106 2 rpy=0 0 0
- joint 1_2: origin xyz=0.7077990772252228 0.4002407024406651 0.4744817559157646 rpy=0 0 0 -> xyz=0.5657439284557486 0.3112542958315417 0.43805783004026333 rpy=0 0 0
- joint 2_3: origin xyz=0.6774918467528679 0.27718605613376096 0.47479675945880684 rpy=0 0 0 -> xyz=0.5837946711273645 0.28685758019741314 0.37198134202571775 rpy=0 0 0
- joint 3_4: origin xyz=0.6886849246465296 0.4689252598316078 0.2986052305643683 rpy=0 0 0 -> xyz=0.9694126675599994 0.4073827757170446 0.3782714453816406 rpy=0 0 0

Commit message: fixed joint and link locations

File: body.urdf (robot description, URDF)
Before this commit: robot robot, 5 links, 4 joints
Links:
- added link 10, mass 0.33013335478447003; collision box size=0.5413929930518149 0.6536675773044348 0.7346559873777192; visual box size=0.5413929930518149 0.6536675773044348 0.7346559873777192
- added link 5, mass 0.4678393086257596; collision box size=0.7084630538268928 0.8853996778352109 0.7458305056092329; visual box size=0.7084630538268928 0.8853996778352109 0.7458305056092329
- added link 6, mass 0.4131154881980677; collision box size=0.9014498957666118 0.5700869075522839 0.8038755457230675; visual box size=0.9014498957666118 0.5700869075522839 0.8038755457230675
- added link 7, mass 0.38373327332077056; collision box size=0.8685681465992023 0.7944575418546873 0.556102526093637; visual box size=0.8685681465992023 0.7944575418546873 0.556102526093637
- added link 8, mass 0.35286575562695904; collision box size=0.667300548085754 0.8007254442223648 0.6603959527791257; visual box size=0.667300548085754 0.8007254442223648 0.6603959527791257
- added link 9, mass 0.33013335478447003; collision box size=0.5406008924539267 0.746609620739366 0.8179355134138371; visual box size=0.5406008924539267 0.746609620739366 0.8179355134138371
- link 0: mass 0.42795200418098583 -> 0.4672596107694953; geometry collision box size=0.9292989366401918 0.663674262784018 0.7576137124535618; visual box size=0.9292989366401918 0.663674262784018 0.7576137124535618
- link 1: mass 0.3085508128028748 -> 0.5021633367710349; geometry collision box size=0.8743065948468078 0.5984717369022319 0.9597046558439345; visual box size=0.8743065948468078 0.5984717369022319 0.9597046558439345
- link 2: mass 0.24917680061749625 -> 0.45762855897014004; geometry collision box size=0.9383224734768658 0.7805730380209224 0.6248092568147998; visual box size=0.9383224734768658 0.7805730380209224 0.6248092568147998
- link 3: mass 0.5975508983060559 -> 0.32955771775091053; geometry collision box size=0.713271039724789 0.6260484033050087 0.7380214480064176; visual box size=0.713271039724789 0.6260484033050087 0.7380214480064176
- link 4: mass 0.5975508983060559 -> 0.5566125293256085; geometry collision box size=0.8938062411872328 0.9066323051661747 0.6868761001619588; visual box size=0.8938062411872328 0.9066323051661747 0.6868761001619588
Joints:
- added joint 4_5: type revolute, parent 4, child 5, origin xyz=0.8938062411872328 0 0 rpy=0 0 0, axis 0 1 0, limit lower=-3.14159 upper=3.14159 effort=0.0 velocity=0.0
- added joint 5_6: type revolute, parent 5, child 6, origin xyz=0.7084630538268928 0 0 rpy=0 0 0, axis 0 1 0, limit lower=-3.14159 upper=3.14159 effort=0.0 velocity=0.0
- added joint 6_7: type revolute, parent 6, child 7, origin xyz=0.9014498957666118 0 0 rpy=0 0 0, axis 0 1 0, limit lower=-3.14159 upper=3.14159 effort=0.0 velocity=0.0
- added joint 7_8: type revolute, parent 7, child 8, origin xyz=0.8685681465992023 0 0 rpy=0 0 0, axis 0 1 0, limit lower=-3.14159 upper=3.14159 effort=0.0 velocity=0.0
- added joint 8_9: type revolute, parent 8, child 9, origin xyz=0.667300548085754 0 0 rpy=0 0 0, axis 0 1 0, limit lower=-3.14159 upper=3.14159 effort=0.0 velocity=0.0
- added joint 9_10: type revolute, parent 9, child 10, origin xyz=0.5406008924539267 0 0 rpy=0 0 0, axis 0 1 0, limit lower=-3.14159 upper=3.14159 effort=0.0 velocity=0.0
- joint 0_1: axis 1 0 0 -> 0 1 0; origin xyz=0.3418030654366779 0.41025366740204106 2 rpy=0 0 0 -> xyz=0.4646494683200959 0 2 rpy=0 0 0
- joint 1_2: axis 1 0 0 -> 0 1 0; origin xyz=0.5657439284557486 0.3112542958315417 0.43805783004026333 rpy=0 0 0 -> xyz=0.8743065948468078 0 0 rpy=0 0 0
- joint 2_3: axis 1 0 0 -> 0 1 0; origin xyz=0.5837946711273645 0.28685758019741314 0.37198134202571775 rpy=0 0 0 -> xyz=0.9383224734768658 0 0 rpy=0 0 0
- joint 3_4: axis 1 0 0 -> 0 1 0; origin xyz=0.9694126675599994 0.4073827757170446 0.3782714453816406 rpy=0 0 0 -> xyz=0.713271039724789 0 0 rpy=0 0 0

Commit message: assign sensor values and colors for links

File: body.urdf (robot description, URDF)
Before this commit: robot robot, 11 links, 10 joints
Links:
- removed link 10
- link 0: mass 0.4672596107694953 -> 0.4211287577313499; geometry collision box size=0.8210303078274538 0.7455850092929881 0.6879526415482403; visual box size=0.8210303078274538 0.7455850092929881 0.6879526415482403
- link 1: mass 0.5021633367710349 -> 0.400487946168033; geometry collision box size=0.6562017770813855 0.7807922384217889 0.7816576085172144; visual box size=0.6562017770813855 0.7807922384217889 0.7816576085172144
- link 2: mass 0.45762855897014004 -> 0.44729053807861646; geometry collision box size=0.7677381895227249 0.7569796517458066 0.7696483835748011; visual box size=0.7677381895227249 0.7569796517458066 0.7696483835748011
- link 3: mass 0.32955771775091053 -> 0.40909059326921615; geometry collision box size=0.5766457172955013 0.8326799283499904 0.8519857407573186; visual box size=0.5766457172955013 0.8326799283499904 0.8519857407573186
- link 4: mass 0.5566125293256085 -> 0.3173228672078326; geometry collision box size=0.6890721015883206 0.886544597443434 0.5194408674789079; visual box size=0.6890721015883206 0.886544597443434 0.5194408674789079
- link 5: mass 0.4678393086257596 -> 0.5388043085012417; geometry collision box size=0.6207002357966499 0.9742568072642841 0.8909958896368388; visual box size=0.6207002357966499 0.9742568072642841 0.8909958896368388
- link 6: mass 0.4131154881980677 -> 0.6933760147810616; geometry collision box size=0.8211097127583937 0.9965482373348644 0.8473626159440635; visual box size=0.8211097127583937 0.9965482373348644 0.8473626159440635
- link 7: mass 0.38373327332077056 -> 0.22648027261892342; geometry collision box size=0.5298220444769071 0.7537801742678627 0.5670947730669256; visual box size=0.5298220444769071 0.7537801742678627 0.5670947730669256
- link 8: mass 0.35286575562695904 -> 0.4176997655307733; geometry collision box size=0.7069015878824707 0.8580852799770098 0.6886123737926949; visual box size=0.7069015878824707 0.8580852799770098 0.6886123737926949
- link 9: mass 0.33013335478447003 -> 0.4176997655307733; geometry collision box size=0.623677745124974 0.8335674252747175 0.6256993476108382; visual box size=0.623677745124974 0.8335674252747175 0.6256993476108382
Joints:
- removed joint 9_10
- joint 0_1: origin xyz=0.4646494683200959 0 2 rpy=0 0 0 -> xyz=0.4105151539137269 0 2 rpy=0 0 0
- joint 1_2: origin xyz=0.8743065948468078 0 0 rpy=0 0 0 -> xyz=0.6562017770813855 0 0 rpy=0 0 0
- joint 2_3: origin xyz=0.9383224734768658 0 0 rpy=0 0 0 -> xyz=0.7677381895227249 0 0 rpy=0 0 0
- joint 3_4: origin xyz=0.713271039724789 0 0 rpy=0 0 0 -> xyz=0.5766457172955013 0 0 rpy=0 0 0
- joint 4_5: origin xyz=0.8938062411872328 0 0 rpy=0 0 0 -> xyz=0.6890721015883206 0 0 rpy=0 0 0
- joint 5_6: origin xyz=0.7084630538268928 0 0 rpy=0 0 0 -> xyz=0.6207002357966499 0 0 rpy=0 0 0
- joint 6_7: origin xyz=0.9014498957666118 0 0 rpy=0 0 0 -> xyz=0.8211097127583937 0 0 rpy=0 0 0
- joint 7_8: origin xyz=0.8685681465992023 0 0 rpy=0 0 0 -> xyz=0.5298220444769071 0 0 rpy=0 0 0
- joint 8_9: origin xyz=0.667300548085754 0 0 rpy=0 0 0 -> xyz=0.7069015878824707 0 0 rpy=0 0 0
