Commit message: made snake body class

File: body.urdf (robot description, URDF)
Before this commit: robot robot, 10 links, 9 joints
Links:
- removed link 7
- removed link 8
- removed link 9
- link 0: mass 0.4211287577313499 -> 0.32618922376833337; geometry collision box size=0.6157136577287 0.9151435049080663 0.5788974284204937; visual box size=0.6157136577287 0.9151435049080663 0.5788974284204937
- link 1: mass 0.400487946168033 -> 0.8449085341419045; geometry collision box size=0.9036675803076387 0.942329453037141 0.9921977306877479; visual box size=0.9036675803076387 0.942329453037141 0.9921977306877479
- link 2: mass 0.44729053807861646 -> 0.2634160360637629; geometry collision box size=0.5662757309423905 0.6992089496932985 0.6652843116242445; visual box size=0.5662757309423905 0.6992089496932985 0.6652843116242445
- link 3: mass 0.40909059326921615 -> 0.37229788590025903; geometry collision box size=0.659269006503092 0.69066417598902 0.8176378370079511; visual box size=0.659269006503092 0.69066417598902 0.8176378370079511
- link 4: mass 0.3173228672078326 -> 0.34501152928579093; geometry collision box size=0.7787527527024977 0.6755786168501645 0.6557799259770052; visual box size=0.7787527527024977 0.6755786168501645 0.6557799259770052
- link 5: mass 0.5388043085012417 -> 0.2967184298022962; geometry collision box size=0.5788819562917713 0.9155069583200445 0.5598773002268784; visual box size=0.5788819562917713 0.9155069583200445 0.5598773002268784
- link 6: mass 0.6933760147810616 -> 0.2767509191575373; geometry collision box size=0.7990954413366621 0.6785195234259745 0.5104204551498219; visual box size=0.7990954413366621 0.6785195234259745 0.5104204551498219
Joints:
- removed joint 6_7
- removed joint 7_8
- removed joint 8_9
- joint 0_1: origin xyz=0.4105151539137269 0 2 rpy=0 0 0 -> xyz=0.30785682886435 0 2 rpy=0 0 0
- joint 1_2: origin xyz=0.6562017770813855 0 0 rpy=0 0 0 -> xyz=0.9036675803076387 0 0 rpy=0 0 0
- joint 2_3: origin xyz=0.7677381895227249 0 0 rpy=0 0 0 -> xyz=0.5662757309423905 0 0 rpy=0 0 0
- joint 3_4: origin xyz=0.5766457172955013 0 0 rpy=0 0 0 -> xyz=0.659269006503092 0 0 rpy=0 0 0
- joint 4_5: origin xyz=0.6890721015883206 0 0 rpy=0 0 0 -> xyz=0.7787527527024977 0 0 rpy=0 0 0
- joint 5_6: origin xyz=0.6207002357966499 0 0 rpy=0 0 0 -> xyz=0.5788819562917713 0 0 rpy=0 0 0

Commit message: make brain neurons and send synapses

File: body.urdf (robot description, URDF)
Before this commit: robot robot, 7 links, 6 joints
Links:
- removed link 0
- removed link 1
- removed link 2
- removed link 3
- removed link 4
- removed link 5
- removed link 6
- added link Link0, mass 0.21624541369894298; collision box size=0.6289843112378013 0.6062558256629118 0.5670889272850883; visual box size=0.6289843112378013 0.6062558256629118 0.5670889272850883
- added link Link1, mass 0.5811824037493866; collision box size=0.9178768330239417 0.8398412137662195 0.7539297228844999; visual box size=0.9178768330239417 0.8398412137662195 0.7539297228844999
- added link Link2, mass 0.5316901750132368; collision box size=0.9644083659141655 0.5847642782086091 0.942794046238755; visual box size=0.9644083659141655 0.5847642782086091 0.942794046238755
- added link Link3, mass 0.18348856189937793; collision box size=0.529387993066008 0.539368021143064 0.642613309427384; visual box size=0.529387993066008 0.539368021143064 0.642613309427384
- added link Link4, mass 0.4901703055930457; collision box size=0.7507298357866078 0.9529532095751408 0.6851595966656147; visual box size=0.7507298357866078 0.9529532095751408 0.6851595966656147
- added link Link5, mass 0.28084461013944767; collision box size=0.6211399637346364 0.8082302805762832 0.559424527511536; visual box size=0.6211399637346364 0.8082302805762832 0.559424527511536
Joints:
- removed joint 0_1
- removed joint 1_2
- removed joint 2_3
- removed joint 3_4
- removed joint 4_5
- removed joint 5_6
- added joint Link0_Link1: type revolute, parent Link0, child Link1, origin xyz=0.31449215561890065 0 2 rpy=0 0 0, axis 0 1 0, limit lower=-3.14159 upper=3.14159 effort=0.0 velocity=0.0
- added joint Link1_Link2: type revolute, parent Link1, child Link2, origin xyz=0.9178768330239417 0 0 rpy=0 0 0, axis 0 1 0, limit lower=-3.14159 upper=3.14159 effort=0.0 velocity=0.0
- added joint Link2_Link3: type revolute, parent Link2, child Link3, origin xyz=0.9644083659141655 0 0 rpy=0 0 0, axis 0 1 0, limit lower=-3.14159 upper=3.14159 effort=0.0 velocity=0.0
- added joint Link3_Link4: type revolute, parent Link3, child Link4, origin xyz=0.529387993066008 0 0 rpy=0 0 0, axis 0 1 0, limit lower=-3.14159 upper=3.14159 effort=0.0 velocity=0.0
- added joint Link4_Link5: type revolute, parent Link4, child Link5, origin xyz=0.7507298357866078 0 0 rpy=0 0 0, axis 0 1 0, limit lower=-3.14159 upper=3.14159 effort=0.0 velocity=0.0

Commit message: fix read me and get everything buttoned up

File: body.urdf (robot description, URDF)
Before this commit: robot robot, 6 links, 5 joints
Links:
- added link Link10, mass 0.3920641807174063; collision box size=1.2398163601364127 1.1891189610311694 0.26593438799682656; visual box size=1.2398163601364127 1.1891189610311694 0.26593438799682656
- added link Link11, mass 0.4898981187686099; collision box size=1.2253906279346132 1.1148420034671513 0.35860628286243346; visual box size=1.2253906279346132 1.1148420034671513 0.35860628286243346
- added link Link6, mass 0.23707409921134104; collision box size=0.9795098964508158 0.37575387189398235 0.6441274634964987; visual box size=0.9795098964508158 0.37575387189398235 0.6441274634964987
- added link Link7, mass 0.8550809426169802; collision box size=1.113583328559884 0.6412291638681 1.1974881941358344; visual box size=1.113583328559884 0.6412291638681 1.1974881941358344
- added link Link8, mass 0.2934778089452228; collision box size=0.4011846772780475 1.018867087194433 0.7179817369440525; visual box size=0.4011846772780475 1.018867087194433 0.7179817369440525
- added link Link9, mass 0.372522327501257; collision box size=1.0563453471614344 0.7882358126730648 0.4473940678202638; visual box size=1.0563453471614344 0.7882358126730648 0.4473940678202638
- link Link0: mass 0.21624541369894298 -> 0.17992568012272867; geometry collision box size=1.0770499529264703 0.45661973585883386 0.3658496369843246; visual box size=1.0770499529264703 0.45661973585883386 0.3658496369843246
- link Link1: mass 0.5811824037493866 -> 0.18947216165102634; geometry collision box size=0.707918169476511 0.5386501754873054 0.4968846095366304; visual box size=0.707918169476511 0.5386501754873054 0.4968846095366304
- link Link2: mass 0.5316901750132368 -> 0.556231181917927; geometry collision box size=0.5395564506496819 1.0465961175012644 0.9850070140034983; visual box size=0.5395564506496819 1.0465961175012644 0.9850070140034983
- link Link3: mass 0.18348856189937793 -> 0.06125189338723071; geometry collision box size=0.5626599077849734 0.3874153060576846 0.2809938225484082; visual box size=0.5626599077849734 0.3874153060576846 0.2809938225484082
- link Link4: mass 0.4901703055930457 -> 0.392512413416429; geometry collision box size=0.4220227012316954 1.2192862726266467 0.7628021331154062; visual box size=0.4220227012316954 1.2192862726266467 0.7628021331154062
- link Link5: mass 0.28084461013944767 -> 0.5020092248169797; geometry collision box size=1.1201850663705506 0.8041939473134051 0.5572641681448881; visual box size=1.1201850663705506 0.8041939473134051 0.5572641681448881
Joints:
- added joint Link10_Link11: type revolute, parent Link10, child Link11, origin xyz=1.2398163601364127 0 0 rpy=0 0 0, axis 0 1 0, limit lower=-3.14159 upper=3.14159 effort=0.0 velocity=0.0
- added joint Link5_Link6: type revolute, parent Link5, child Link6, origin xyz=1.1201850663705506 0 0 rpy=0 0 0, axis 0 1 0, limit lower=-3.14159 upper=3.14159 effort=0.0 velocity=0.0
- added joint Link6_Link7: type revolute, parent Link6, child Link7, origin xyz=0.9795098964508158 0 0 rpy=0 0 0, axis 0 1 0, limit lower=-3.14159 upper=3.14159 effort=0.0 velocity=0.0
- added joint Link7_Link8: type revolute, parent Link7, child Link8, origin xyz=1.113583328559884 0 0 rpy=0 0 0, axis 0 1 0, limit lower=-3.14159 upper=3.14159 effort=0.0 velocity=0.0
- added joint Link8_Link9: type revolute, parent Link8, child Link9, origin xyz=0.4011846772780475 0 0 rpy=0 0 0, axis 0 1 0, limit lower=-3.14159 upper=3.14159 effort=0.0 velocity=0.0
- added joint Link9_Link10: type revolute, parent Link9, child Link10, origin xyz=1.0563453471614344 0 0 rpy=0 0 0, axis 0 1 0, limit lower=-3.14159 upper=3.14159 effort=0.0 velocity=0.0
- joint Link0_Link1: origin xyz=0.31449215561890065 0 2 rpy=0 0 0 -> xyz=0.5385249764632352 0 2 rpy=0 0 0
- joint Link1_Link2: origin xyz=0.9178768330239417 0 0 rpy=0 0 0 -> xyz=0.707918169476511 0 0 rpy=0 0 0
- joint Link2_Link3: origin xyz=0.9644083659141655 0 0 rpy=0 0 0 -> xyz=0.5395564506496819 0 0 rpy=0 0 0
- joint Link3_Link4: origin xyz=0.529387993066008 0 0 rpy=0 0 0 -> xyz=0.5626599077849734 0 0 rpy=0 0 0
- joint Link4_Link5: origin xyz=0.7507298357866078 0 0 rpy=0 0 0 -> xyz=0.4220227012316954 0 0 rpy=0 0 0

Commit message: Finish making body and updating README

File: body.urdf (robot description, URDF)
Before this commit: robot robot, 12 links, 11 joints
Links:
- removed link Link10
- removed link Link11
- removed link Link5
- removed link Link6
- removed link Link7
- removed link Link8
- removed link Link9
- link Link0: mass 0.17992568012272867 -> 0.11972454002546074; geometry collision box size=0.25871069360547383 0.9206225209371665 0.5026749022649195; visual box size=0.25871069360547383 0.9206225209371665 0.5026749022649195
- link Link1: mass 0.18947216165102634 -> 0.24237794987561107; geometry collision box size=0.816761627627743 0.4916643869011911 0.6035719242869888; visual box size=0.816761627627743 0.4916643869011911 0.6035719242869888
- link Link2: mass 0.556231181917927 -> 0.6476432602566873; geometry collision box size=0.9552384454927307 0.724292253873224 0.9360740732761972; visual box size=0.9552384454927307 0.724292253873224 0.9360740732761972
- link Link3: mass 0.06125189338723071 -> 0.10385285125339688; geometry collision box size=0.7211534253924048 0.5238273978029255 0.2749176001455893; visual box size=0.7211534253924048 0.5238273978029255 0.2749176001455893
- link Link4: mass 0.392512413416429 -> 0.08702582501996244; geometry collision box size=0.4314501846220483 0.7442613129634019 0.2710141991100593; visual box size=0.4314501846220483 0.7442613129634019 0.2710141991100593
Joints:
- removed joint Link10_Link11
- removed joint Link4_Link5
- removed joint Link5_Link6
- removed joint Link6_Link7
- removed joint Link7_Link8
- removed joint Link8_Link9
- removed joint Link9_Link10
- joint Link0_Link1: axis 0 1 0 -> 1 0 0; origin xyz=0.5385249764632352 0 2 rpy=0 0 0 -> xyz=0.12935534680273691 0 2 rpy=0 0 0
- joint Link1_Link2: origin xyz=0.707918169476511 0 0 rpy=0 0 0 -> xyz=0.4083808138138715 0.0 -0.3017859621434944 rpy=0 0 0
- joint Link2_Link3: axis 0 1 0 -> 1 0 0; origin xyz=0.5395564506496819 0 0 rpy=0 0 0 -> xyz=0.0 0.0 -0.9360740732761972 rpy=0 0 0
- joint Link3_Link4: axis 0 1 0 -> 0 0 1; origin xyz=0.5626599077849734 0 0 rpy=0 0 0 -> xyz=0.3605767126962024 0.0 -0.13745880007279465 rpy=0 0 0

Commit message: Begin setting up checkpointing and random seed

File: body.urdf (robot description, URDF)
Before this commit: robot robot, 5 links, 4 joints
Links:
- added link Link5, mass 0.2100501022568541; collision box size=0.6606558803776915 1.1394983248528585 0.27901907929990444; visual box size=0.6606558803776915 1.1394983248528585 0.27901907929990444
- added link Link6, mass 0.8518180446761869; collision box size=1.1102341537871503 0.696624299889673 1.101370989800485; visual box size=1.1102341537871503 0.696624299889673 1.101370989800485
- added link Link7, mass 0.3239948402140874; collision box size=0.8763494817410246 1.0406627525510057 0.3552636301430251; visual box size=0.8763494817410246 1.0406627525510057 0.3552636301430251
- added link Link8, mass 0.5173387455830804; collision box size=1.0668929376424992 0.41881415354060825 1.1577980544452684; visual box size=1.0668929376424992 0.41881415354060825 1.1577980544452684
- added link Link9, mass 0.13070028714317322; collision box size=0.7300050043380578 0.5821969346649141 0.3075252568499913; visual box size=0.7300050043380578 0.5821969346649141 0.3075252568499913
- link Link0: mass 0.11972454002546074 -> 0.2764667265180527; geometry collision box size=1.12668761676496 0.7923106238756858 0.3097019001489896; visual box size=1.12668761676496 0.7923106238756858 0.3097019001489896
- link Link1: mass 0.24237794987561107 -> 0.09221813343197821; geometry collision box size=0.9508975203366635 0.29056921473672004 0.3337590210430188; visual box size=0.9508975203366635 0.29056921473672004 0.3337590210430188
- link Link2: mass 0.6476432602566873 -> 0.18803913065462094; geometry collision box size=0.3250328573054725 0.5731329761373101 1.0094052797311401; visual box size=0.3250328573054725 0.5731329761373101 1.0094052797311401
- link Link3: mass 0.10385285125339688 -> 0.3062921745620059; geometry collision box size=0.5548003426591548 0.5101040743133963 1.0822818820692364; visual box size=0.5548003426591548 0.5101040743133963 1.0822818820692364
- link Link4: mass 0.08702582501996244 -> 0.12749826005242026; geometry collision box size=0.30958108873478096 0.6002808570747119 0.6860809186956035; visual box size=0.30958108873478096 0.6002808570747119 0.6860809186956035
Joints:
- added joint Link4_Link5: type revolute, parent Link4, child Link5, origin xyz=0.0 -0.6002808570747119 0.0 rpy=0 0 0, axis 1 0 0, limit lower=-3.14159 upper=3.14159 effort=0.0 velocity=0.0
- added joint Link5_Link6: type revolute, parent Link5, child Link6, origin xyz=0.0 -0.5697491624264293 -0.13950953964995222 rpy=0 0 0, axis 0 1 0, limit lower=-3.14159 upper=3.14159 effort=0.0 velocity=0.0
- added joint Link6_Link7: type revolute, parent Link6, child Link7, origin xyz=0.0 -0.3483121499448365 -0.5506854949002425 rpy=0 0 0, axis 0 0 1, limit lower=-3.14159 upper=3.14159 effort=0.0 velocity=0.0
- added joint Link7_Link8: type revolute, parent Link7, child Link8, origin xyz=0.4381747408705123 -0.5203313762755029 0.0 rpy=0 0 0, axis 0 0 1, limit lower=-3.14159 upper=3.14159 effort=0.0 velocity=0.0
- added joint Link8_Link9: type revolute, parent Link8, child Link9, origin xyz=0.5334464688212496 0.0 0.5788990272226342 rpy=0 0 0, axis 1 0 0, limit lower=-3.14159 upper=3.14159 effort=0.0 velocity=0.0
- joint Link0_Link1: origin xyz=0.12935534680273691 0 2 rpy=0 0 0 -> xyz=0.56334380838248 0 2 rpy=0 0 0
- joint Link1_Link2: origin xyz=0.4083808138138715 0.0 -0.3017859621434944 rpy=0 0 0 -> xyz=0.47544876016833176 -0.14528460736836002 0.0 rpy=0 0 0
- joint Link2_Link3: axis 1 0 0 -> 0 1 0; origin xyz=0.0 0.0 -0.9360740732761972 rpy=0 0 0 -> xyz=0.0 -0.5731329761373101 0.0 rpy=0 0 0
- joint Link3_Link4: axis 0 0 1 -> 1 0 0; origin xyz=0.3605767126962024 0.0 -0.13745880007279465 rpy=0 0 0 -> xyz=0.0 -0.5101040743133963 0.0 rpy=0 0 0

Commit message: Random Seeding working

File: body.urdf (robot description, URDF)
Before this commit: robot robot, 10 links, 9 joints
Links:
- link Link0: mass 0.2764667265180527 -> 1.1863161466101886; geometry collision box size=1.2170298390136767 0.7972322491757223 1.2226843599648842; visual box size=1.2170298390136767 0.7972322491757223 1.2226843599648842
- link Link1: mass 0.09221813343197821 -> 0.24159438313137246; geometry collision box size=0.4719931710897395 1.1207323061773764 0.4567191553394264; visual box size=0.4719931710897395 1.1207323061773764 0.4567191553394264
- link Link2: mass 0.18803913065462094 -> 0.7124975516153823; geometry collision box size=1.1428601514360017 0.5819798053011772 1.0712291230578317; visual box size=1.1428601514360017 0.5819798053011772 1.0712291230578317
- link Link3: mass 0.3062921745620059 -> 0.23135440586714634; geometry collision box size=0.32630828937395717 1.0299187922401147 0.6884092314408935; visual box size=0.32630828937395717 1.0299187922401147 0.6884092314408935
- link Link4: mass 0.12749826005242026 -> 1.5321151085328013; geometry collision box size=1.1234294027918161 1.2185406628209319 1.11919454021392; visual box size=1.1234294027918161 1.2185406628209319 1.11919454021392
- link Link5: mass 0.2100501022568541 -> 0.14599907611527876; geometry collision box size=0.26037415388569995 0.7518745921487388 0.7457732931341461; visual box size=0.26037415388569995 0.7518745921487388 0.7457732931341461
- link Link6: mass 0.8518180446761869 -> 0.2443504350150486; geometry collision box size=1.0213206432667459 0.2707519493594015 0.8836482349262754; visual box size=1.0213206432667459 0.2707519493594015 0.8836482349262754
- link Link7: mass 0.3239948402140874 -> 0.0826955686865952; geometry collision box size=0.4302696888767692 0.2694752414876246 0.7132185264983446; visual box size=0.4302696888767692 0.2694752414876246 0.7132185264983446
- link Link8: mass 0.5173387455830804 -> 0.20539853719865275; geometry collision box size=0.40416284237967237 0.9900496965154048 0.5133150151851347; visual box size=0.40416284237967237 0.9900496965154048 0.5133150151851347
- link Link9: mass 0.13070028714317322 -> 0.5382643443625381; geometry collision box size=1.0277024105738202 0.4875412200349123 1.0742785326613684; visual box size=1.0277024105738202 0.4875412200349123 1.0742785326613684
Joints:
- joint Link0_Link1: origin xyz=0.56334380838248 0 2 rpy=0 0 0 -> xyz=0.6085149195068383 0 2 rpy=0 0 0
- joint Link1_Link2: axis 0 1 0 -> 0 0 1; origin xyz=0.47544876016833176 -0.14528460736836002 0.0 rpy=0 0 0 -> xyz=0.4719931710897395 0.0 0.0 rpy=0 0 0
- joint Link2_Link3: axis 0 1 0 -> 0 0 1; origin xyz=0.0 -0.5731329761373101 0.0 rpy=0 0 0 -> xyz=1.1428601514360017 0.0 0.0 rpy=0 0 0
- joint Link3_Link4: axis 1 0 0 -> 0 1 0; origin xyz=0.0 -0.5101040743133963 0.0 rpy=0 0 0 -> xyz=0.16315414468697859 0.5149593961200574 0.0 rpy=0 0 0
- joint Link4_Link5: origin xyz=0.0 -0.6002808570747119 0.0 rpy=0 0 0 -> xyz=0.0 1.2185406628209319 0.0 rpy=0 0 0
- joint Link5_Link6: origin xyz=0.0 -0.5697491624264293 -0.13950953964995222 rpy=0 0 0 -> xyz=0.0 0.7518745921487388 0.0 rpy=0 0 0
- joint Link6_Link7: origin xyz=0.0 -0.3483121499448365 -0.5506854949002425 rpy=0 0 0 -> xyz=0.0 0.13537597467970075 0.4418241174631377 rpy=0 0 0
- joint Link7_Link8: axis 0 0 1 -> 0 1 0; origin xyz=0.4381747408705123 -0.5203313762755029 0.0 rpy=0 0 0 -> xyz=0.0 0.1347376207438123 0.3566092632491723 rpy=0 0 0
- joint Link8_Link9: axis 1 0 0 -> 0 1 0; origin xyz=0.5334464688212496 0.0 0.5788990272226342 rpy=0 0 0 -> xyz=0.0 0.9900496965154048 0.0 rpy=0 0 0

Commit message: Moved the weights initialization to create snake brain

File: body.urdf (robot description, URDF)
Before this commit: robot robot, 10 links, 9 joints
Links:
- link Link0: mass 1.1863161466101886 -> 0.16188097376707722; geometry collision box size=0.667022004702574 0.9703244934421581 0.2501143748173449; visual box size=0.667022004702574 0.9703244934421581 0.2501143748173449
- link Link1: mass 0.24159438313137246 -> 0.15136330318765737; geometry collision box size=0.6859949021420038 0.27592623182789133 0.7996624778787091; visual box size=0.6859949021420038 0.27592623182789133 0.7996624778787091
- link Link2: mass 0.7124975516153823 -> 0.41502688459911957; geometry collision box size=0.8007979025745755 0.9581478226181048 0.5409047389129443; visual box size=0.8007979025745755 0.9581478226181048 0.5409047389129443
- link Link3: mass 0.23135440586714634 -> 1.1863161466101886; geometry collision box size=1.2170298390136767 0.7972322491757223 1.2226843599648842; visual box size=1.2170298390136767 0.7972322491757223 1.2226843599648842
- link Link4: mass 1.5321151085328013 -> 0.24159438313137246; geometry collision box size=0.4719931710897395 1.1207323061773764 0.4567191553394264; visual box size=0.4719931710897395 1.1207323061773764 0.4567191553394264
- link Link5: mass 0.14599907611527876 -> 0.7124975516153823; geometry collision box size=1.1428601514360017 0.5819798053011772 1.0712291230578317; visual box size=1.1428601514360017 0.5819798053011772 1.0712291230578317
- link Link6: mass 0.2443504350150486 -> 0.23135440586714634; geometry collision box size=0.32630828937395717 1.0299187922401147 0.6884092314408935; visual box size=0.32630828937395717 1.0299187922401147 0.6884092314408935
- link Link7: mass 0.0826955686865952 -> 1.5321151085328013; geometry collision box size=1.1234294027918161 1.2185406628209319 1.11919454021392; visual box size=1.1234294027918161 1.2185406628209319 1.11919454021392
- link Link8: mass 0.20539853719865275 -> 0.14599907611527876; geometry collision box size=0.26037415388569995 0.7518745921487388 0.7457732931341461; visual box size=0.26037415388569995 0.7518745921487388 0.7457732931341461
- link Link9: mass 0.5382643443625381 -> 0.2443504350150486; geometry collision box size=1.0213206432667459 0.2707519493594015 0.8836482349262754; visual box size=1.0213206432667459 0.2707519493594015 0.8836482349262754
Joints:
- joint Link0_Link1: origin xyz=0.6085149195068383 0 2 rpy=0 0 0 -> xyz=0.333511002351287 0 2 rpy=0 0 0
- joint Link1_Link2: axis 0 0 1 -> 1 0 0; origin xyz=0.4719931710897395 0.0 0.0 rpy=0 0 0 -> xyz=0.3429974510710019 -0.13796311591394567 0.0 rpy=0 0 0
- joint Link2_Link3: axis 0 0 1 -> 1 0 0; origin xyz=1.1428601514360017 0.0 0.0 rpy=0 0 0 -> xyz=-0.40039895128728775 -0.4790739113090524 0.0 rpy=0 0 0
- joint Link3_Link4: axis 0 1 0 -> 1 0 0; origin xyz=0.16315414468697859 0.5149593961200574 0.0 rpy=0 0 0 -> xyz=-0.6085149195068383 -0.39861612458786116 0.0 rpy=0 0 0
- joint Link4_Link5: axis 1 0 0 -> 0 0 1; origin xyz=0.0 1.2185406628209319 0.0 rpy=0 0 0 -> xyz=-0.23599658554486974 -0.5603661530886882 0.0 rpy=0 0 0
- joint Link5_Link6: axis 0 1 0 -> 0 0 1; origin xyz=0.0 0.7518745921487388 0.0 rpy=0 0 0 -> xyz=-0.5714300757180009 -0.2909899026505886 0.0 rpy=0 0 0
- joint Link6_Link7: axis 0 0 1 -> 0 1 0; origin xyz=0.0 0.13537597467970075 0.4418241174631377 rpy=0 0 0 -> xyz=0.0 -1.0299187922401147 0.0 rpy=0 0 0
- joint Link7_Link8: axis 0 1 0 -> 1 0 0; origin xyz=0.0 0.1347376207438123 0.3566092632491723 rpy=0 0 0 -> xyz=0.5617147013959081 -0.6092703314104659 0.0 rpy=0 0 0
- joint Link8_Link9: origin xyz=0.0 0.9900496965154048 0.0 rpy=0 0 0 -> xyz=0.13018707694284998 0.3759372960743694 0.0 rpy=0 0 0
