Commit message: Getting ready to run for each of the selected bodies

File: body0.urdf (robot description, URDF)
Before this commit: robot robot, 10 links, 9 joints
Links:
- link Link0: mass 0.16188097376707722 -> 0.24159438313137246; geometry collision box size=0.4719931710897395 1.1207323061773764 0.4567191553394264; visual box size=0.4719931710897395 1.1207323061773764 0.4567191553394264
- link Link1: mass 0.15136330318765737 -> 0.7124975516153823; geometry collision box size=1.1428601514360017 0.5819798053011772 1.0712291230578317; visual box size=1.1428601514360017 0.5819798053011772 1.0712291230578317
- link Link2: mass 0.41502688459911957 -> 0.23135440586714634; geometry collision box size=0.32630828937395717 1.0299187922401147 0.6884092314408935; visual box size=0.32630828937395717 1.0299187922401147 0.6884092314408935
- link Link3: mass 1.1863161466101886 -> 1.5321151085328013; geometry collision box size=1.1234294027918161 1.2185406628209319 1.11919454021392; visual box size=1.1234294027918161 1.2185406628209319 1.11919454021392
- link Link4: mass 0.24159438313137246 -> 0.14599907611527876; geometry collision box size=0.26037415388569995 0.7518745921487388 0.7457732931341461; visual box size=0.26037415388569995 0.7518745921487388 0.7457732931341461
- link Link5: mass 0.7124975516153823 -> 0.2443504350150486; geometry collision box size=1.0213206432667459 0.2707519493594015 0.8836482349262754; visual box size=1.0213206432667459 0.2707519493594015 0.8836482349262754
- link Link6: mass 0.23135440586714634 -> 0.0826955686865952; geometry collision box size=0.4302696888767692 0.2694752414876246 0.7132185264983446; visual box size=0.4302696888767692 0.2694752414876246 0.7132185264983446
- link Link7: mass 1.5321151085328013 -> 0.20539853719865275; geometry collision box size=0.40416284237967237 0.9900496965154048 0.5133150151851347; visual box size=0.40416284237967237 0.9900496965154048 0.5133150151851347
- link Link8: mass 0.14599907611527876 -> 0.5382643443625381; geometry collision box size=1.0277024105738202 0.4875412200349123 1.0742785326613684; visual box size=1.0277024105738202 0.4875412200349123 1.0742785326613684
- link Link9: mass 0.2443504350150486 -> 0.8757712431768542; geometry collision box size=0.7639433437726902 1.0231650520792968 1.1204276857248128; visual box size=0.7639433437726902 1.0231650520792968 1.1204276857248128
Joints:
- joint Link0_Link1: origin xyz=0.333511002351287 0 2 rpy=0 0 0 -> xyz=0.23599658554486974 0 2 rpy=0 0 0
- joint Link1_Link2: axis 1 0 0 -> 0 0 1; origin xyz=0.3429974510710019 -0.13796311591394567 0.0 rpy=0 0 0 -> xyz=0.5714300757180009 0.0 -0.5356145615289158 rpy=0 0 0
- joint Link2_Link3: axis 1 0 0 -> 0 1 0; origin xyz=-0.40039895128728775 -0.4790739113090524 0.0 rpy=0 0 0 -> xyz=0.0 -0.5149593961200574 -0.34420461572044675 rpy=0 0 0
- joint Link3_Link4: origin xyz=-0.6085149195068383 -0.39861612458786116 0.0 rpy=0 0 0 -> xyz=0.0 -0.6092703314104659 0.55959727010696 rpy=0 0 0
- joint Link4_Link5: axis 0 0 1 -> 0 1 0; origin xyz=-0.23599658554486974 -0.5603661530886882 0.0 rpy=0 0 0 -> xyz=0.0 0.3759372960743694 0.37288664656707304 rpy=0 0 0
- joint Link5_Link6: origin xyz=-0.5714300757180009 -0.2909899026505886 0.0 rpy=0 0 0 -> xyz=0.0 0.13537597467970075 -0.4418241174631377 rpy=0 0 0
- joint Link6_Link7: origin xyz=0.0 -1.0299187922401147 0.0 rpy=0 0 0 -> xyz=0.0 0.1347376207438123 -0.3566092632491723 rpy=0 0 0
- joint Link7_Link8: axis 1 0 0 -> 0 1 0; origin xyz=0.5617147013959081 -0.6092703314104659 0.0 rpy=0 0 0 -> xyz=0.0 0.9900496965154048 0.0 rpy=0 0 0
- joint Link8_Link9: origin xyz=0.13018707694284998 0.3759372960743694 0.0 rpy=0 0 0 -> xyz=0.5138512052869101 0.24377061001745615 0.0 rpy=0 0 0

Commit message: Ready to begin simulations for seed 5

File: body0.urdf (robot description, URDF)
Before this commit: robot robot, 10 links, 9 joints
Links:
- link Link0: mass 0.24159438313137246 -> 0.48289623937059023; geometry collision box size=0.5374797485527598 0.9512196524779869 0.9445194457665361; visual box size=0.5374797485527598 0.9512196524779869 0.9445194457665361
- link Link1: mass 0.7124975516153823 -> 0.1740536113612289; geometry collision box size=0.9008498451531076 0.5772149747430876 0.33472876946214414; visual box size=0.9008498451531076 0.5772149747430876 0.33472876946214414
- link Link2: mass 0.23135440586714634 -> 0.6554020118868491; geometry collision box size=1.0002408225691506 0.8358698084045144 0.7839070243994751; visual box size=1.0002408225691506 0.8358698084045144 0.7839070243994751
- link Link3: mass 1.5321151085328013 -> 1.4291587234543774; geometry collision box size=1.0542439692962855 1.150366215625144 1.1784284544657466; visual box size=1.0542439692962855 1.150366215625144 1.1784284544657466
- link Link4: mass 0.14599907611527876 -> 0.3643458102596293; geometry collision box size=0.4014603790841491 1.0017263034512394 0.9059870953742684; visual box size=0.4014603790841491 1.0017263034512394 0.9059870953742684
- link Link5: mass 0.2443504350150486 -> 0.20349246603893198; geometry collision box size=1.0925032911606163 0.3604069977379858 0.5168117346816321; visual box size=1.0925032911606163 0.3604069977379858 0.5168117346816321
- link Link6: mass 0.0826955686865952 -> 0.17827922579545694; geometry collision box size=1.1406231845687314 0.5368183035830643 0.2911596772003453; visual box size=1.1406231845687314 0.5368183035830643 0.2911596772003453
- link Link7: mass 0.20539853719865275 -> 0.3171794428637607; geometry collision box size=1.0576430736828655 0.35111281885189227 0.8541206399752443; visual box size=1.0576430736828655 0.35111281885189227 0.8541206399752443
- link Link8: mass 0.5382643443625381 -> 0.14074526606575816; geometry collision box size=0.7564950724895487 0.38808839948406193 0.47939889821699533; visual box size=0.7564950724895487 0.38808839948406193 0.47939889821699533
- link Link9: mass 0.8757712431768542 -> 0.15612571378956822; geometry collision box size=0.36402197699886896 0.8721124443249966 0.4917839483200783; visual box size=0.36402197699886896 0.8721124443249966 0.4917839483200783
Joints:
- joint Link0_Link1: origin xyz=0.23599658554486974 0 2 rpy=0 0 0 -> xyz=0.2687398742763799 0 2 rpy=0 0 0
- joint Link1_Link2: axis 0 0 1 -> 1 0 0; origin xyz=0.5714300757180009 0.0 -0.5356145615289158 rpy=0 0 0 -> xyz=0.4504249225765538 0.0 0.16736438473107207 rpy=0 0 0
- joint Link2_Link3: axis 0 1 0 -> 0 0 1; origin xyz=0.0 -0.5149593961200574 -0.34420461572044675 rpy=0 0 0 -> xyz=0.0 -0.4179349042022572 0.39195351219973756 rpy=0 0 0
- joint Link3_Link4: axis 1 0 0 -> 0 1 0; origin xyz=0.0 -0.6092703314104659 0.55959727010696 rpy=0 0 0 -> xyz=0.0 -0.575183107812572 0.5892142272328733 rpy=0 0 0
- joint Link4_Link5: origin xyz=0.0 0.3759372960743694 0.37288664656707304 rpy=0 0 0 -> xyz=0.0 0.5008631517256197 0.4529935476871342 rpy=0 0 0
- joint Link5_Link6: axis 0 0 1 -> 1 0 0; origin xyz=0.0 0.13537597467970075 -0.4418241174631377 rpy=0 0 0 -> xyz=-0.5462516455803081 0.1802034988689929 0.0 rpy=0 0 0
- joint Link6_Link7: origin xyz=0.0 0.1347376207438123 -0.3566092632491723 rpy=0 0 0 -> xyz=-0.5703115922843657 -0.26840915179153213 0.0 rpy=0 0 0
- joint Link7_Link8: origin xyz=0.0 0.9900496965154048 0.0 rpy=0 0 0 -> xyz=0.0 -0.35111281885189227 0.0 rpy=0 0 0
- joint Link8_Link9: origin xyz=0.5138512052869101 0.24377061001745615 0.0 rpy=0 0 0 -> xyz=0.0 -0.38808839948406193 0.0 rpy=0 0 0

Commit message: finish 4th simulation

File: body0.urdf (robot description, URDF)
Before this commit: robot robot, 10 links, 9 joints
Links:
- link Link0: mass 0.48289623937059023 -> 0.4431323837220064; geometry collision box size=0.7214481228701298 0.7974544776358078 0.7702336361563769; visual box size=0.7214481228701298 0.7974544776358078 0.7702336361563769
- link Link1: mass 0.1740536113612289 -> 0.27155458959106615; geometry collision box size=0.9251573453988623 0.4631389265762489 0.6337679329684967; visual box size=0.9251573453988623 0.4631389265762489 0.6337679329684967
- link Link2: mass 0.6554020118868491 -> 0.4434412732531254; geometry collision box size=0.5644082047245251 1.1745629989172475 0.6689081363643288; visual box size=0.5644082047245251 1.1745629989172475 0.6689081363643288
- link Link3: mass 1.4291587234543774 -> 0.8007249056108289; geometry collision box size=0.5663231481664555 1.132878372926637 1.248060784448033; visual box size=0.5663231481664555 1.132878372926637 1.248060784448033
- link Link4: mass 0.3643458102596293 -> 0.7966482754225184; geometry collision box size=1.1303299626455037 1.1884984734941606 0.5930110037438258; visual box size=1.1303299626455037 1.1884984734941606 0.5930110037438258
- link Link5: mass 0.20349246603893198 -> 0.8116550952069246; geometry collision box size=1.1268634486504114 0.7116031693251716 1.012190725057534; visual box size=1.1268634486504114 0.7116031693251716 1.012190725057534
- link Link6: mass 0.17827922579545694 -> 0.09201515189415578; geometry collision box size=0.28672935755187545 0.8887680860361484 0.36107609271623675; visual box size=0.28672935755187545 0.8887680860361484 0.36107609271623675
- link Link7: mass 0.3171794428637607 -> 1.1605168132256056; geometry collision box size=0.9883023498001428 1.0800838652009106 1.087186698827849; visual box size=0.9883023498001428 1.0800838652009106 1.087186698827849
- link Link8: mass 0.14074526606575816 -> 0.3784993316948017; geometry collision box size=1.239516946534479 0.4460892653320435 0.6845274616719605; visual box size=1.239516946534479 0.4460892653320435 0.6845274616719605
- link Link9: mass 0.15612571378956822 -> 0.3217161997263615; geometry collision box size=0.6290809782474991 0.5448593425054197 0.9386030789259829; visual box size=0.6290809782474991 0.5448593425054197 0.9386030789259829
Joints:
- joint Link0_Link1: origin xyz=0.2687398742763799 0 2 rpy=0 0 0 -> xyz=0.3607240614350649 0 2 rpy=0 0 0
- joint Link1_Link2: axis 1 0 0 -> 0 1 0; origin xyz=0.4504249225765538 0.0 0.16736438473107207 rpy=0 0 0 -> xyz=0.46257867269943115 0.23156946328812444 0.0 rpy=0 0 0
- joint Link2_Link3: axis 0 0 1 -> 0 1 0; origin xyz=0.0 -0.4179349042022572 0.39195351219973756 rpy=0 0 0 -> xyz=0.0 0.5872814994586237 -0.3344540681821644 rpy=0 0 0
- joint Link3_Link4: axis 0 1 0 -> 1 0 0; origin xyz=0.0 -0.575183107812572 0.5892142272328733 rpy=0 0 0 -> xyz=-0.28316157408322773 0.0 -0.6240303922240165 rpy=0 0 0
- joint Link4_Link5: axis 0 1 0 -> 1 0 0; origin xyz=0.0 0.5008631517256197 0.4529935476871342 rpy=0 0 0 -> xyz=-0.5651649813227518 0.0 0.2965055018719129 rpy=0 0 0
- joint Link5_Link6: axis 1 0 0 -> 0 1 0; origin xyz=-0.5462516455803081 0.1802034988689929 0.0 rpy=0 0 0 -> xyz=0.0 -0.3558015846625858 0.506095362528767 rpy=0 0 0
- joint Link6_Link7: origin xyz=-0.5703115922843657 -0.26840915179153213 0.0 rpy=0 0 0 -> xyz=0.0 -0.4443840430180742 0.18053804635811838 rpy=0 0 0
- joint Link7_Link8: axis 0 1 0 -> 1 0 0; origin xyz=0.0 -0.35111281885189227 0.0 rpy=0 0 0 -> xyz=-0.4941511749000714 0.0 0.5435933494139245 rpy=0 0 0
- joint Link8_Link9: axis 0 1 0 -> 0 0 1; origin xyz=0.0 -0.38808839948406193 0.0 rpy=0 0 0 -> xyz=-0.6197584732672395 0.22304463266602176 0.0 rpy=0 0 0

Commit message: Finish 5th simulation

File: body0.urdf (robot description, URDF)
Before this commit: robot robot, 10 links, 9 joints
Links:
- link Link0: mass 0.4431323837220064 -> 0.16188097376707722; geometry collision box size=0.667022004702574 0.9703244934421581 0.2501143748173449; visual box size=0.667022004702574 0.9703244934421581 0.2501143748173449
- link Link1: mass 0.27155458959106615 -> 0.15136330318765737; geometry collision box size=0.6859949021420038 0.27592623182789133 0.7996624778787091; visual box size=0.6859949021420038 0.27592623182789133 0.7996624778787091
- link Link2: mass 0.4434412732531254 -> 0.41502688459911957; geometry collision box size=0.8007979025745755 0.9581478226181048 0.5409047389129443; visual box size=0.8007979025745755 0.9581478226181048 0.5409047389129443
- link Link3: mass 0.8007249056108289 -> 1.1863161466101886; geometry collision box size=1.2170298390136767 0.7972322491757223 1.2226843599648842; visual box size=1.2170298390136767 0.7972322491757223 1.2226843599648842
- link Link4: mass 0.7966482754225184 -> 0.24159438313137246; geometry collision box size=0.4719931710897395 1.1207323061773764 0.4567191553394264; visual box size=0.4719931710897395 1.1207323061773764 0.4567191553394264
- link Link5: mass 0.8116550952069246 -> 0.7124975516153823; geometry collision box size=1.1428601514360017 0.5819798053011772 1.0712291230578317; visual box size=1.1428601514360017 0.5819798053011772 1.0712291230578317
- link Link6: mass 0.09201515189415578 -> 0.23135440586714634; geometry collision box size=0.32630828937395717 1.0299187922401147 0.6884092314408935; visual box size=0.32630828937395717 1.0299187922401147 0.6884092314408935
- link Link7: mass 1.1605168132256056 -> 1.5321151085328013; geometry collision box size=1.1234294027918161 1.2185406628209319 1.11919454021392; visual box size=1.1234294027918161 1.2185406628209319 1.11919454021392
- link Link8: mass 0.3784993316948017 -> 0.14599907611527876; geometry collision box size=0.26037415388569995 0.7518745921487388 0.7457732931341461; visual box size=0.26037415388569995 0.7518745921487388 0.7457732931341461
- link Link9: mass 0.3217161997263615 -> 0.2443504350150486; geometry collision box size=1.0213206432667459 0.2707519493594015 0.8836482349262754; visual box size=1.0213206432667459 0.2707519493594015 0.8836482349262754
Joints:
- joint Link0_Link1: origin xyz=0.3607240614350649 0 2 rpy=0 0 0 -> xyz=0.333511002351287 0 2 rpy=0 0 0
- joint Link1_Link2: axis 0 1 0 -> 1 0 0; origin xyz=0.46257867269943115 0.23156946328812444 0.0 rpy=0 0 0 -> xyz=0.3429974510710019 -0.13796311591394567 0.0 rpy=0 0 0
- joint Link2_Link3: axis 0 1 0 -> 1 0 0; origin xyz=0.0 0.5872814994586237 -0.3344540681821644 rpy=0 0 0 -> xyz=0.0 -0.4790739113090524 0.27045236945647216 rpy=0 0 0
- joint Link3_Link4: origin xyz=-0.28316157408322773 0.0 -0.6240303922240165 rpy=0 0 0 -> xyz=0.0 0.0 1.2226843599648842 rpy=0 0 0
- joint Link4_Link5: axis 1 0 0 -> 0 0 1; origin xyz=-0.5651649813227518 0.0 0.2965055018719129 rpy=0 0 0 -> xyz=0.0 -0.5603661530886882 0.2283595776697132 rpy=0 0 0
- joint Link5_Link6: axis 0 1 0 -> 0 0 1; origin xyz=0.0 -0.3558015846625858 0.506095362528767 rpy=0 0 0 -> xyz=0.0 -0.2909899026505886 -0.5356145615289158 rpy=0 0 0
- joint Link6_Link7: origin xyz=0.0 -0.4443840430180742 0.18053804635811838 rpy=0 0 0 -> xyz=0.0 -0.5149593961200574 -0.34420461572044675 rpy=0 0 0
- joint Link7_Link8: origin xyz=-0.4941511749000714 0.0 0.5435933494139245 rpy=0 0 0 -> xyz=0.0 -0.6092703314104659 0.55959727010696 rpy=0 0 0
- joint Link8_Link9: axis 0 0 1 -> 0 1 0; origin xyz=-0.6197584732672395 0.22304463266602176 0.0 rpy=0 0 0 -> xyz=0.0 0.3759372960743694 0.37288664656707304 rpy=0 0 0

Commit message: Ready to run final project sims

File: body0.urdf (robot description, URDF)
Before this commit: robot robot, 10 links, 9 joints
Links:
- link Link0: mass 0.16188097376707722 -> 0.32949792017734864; geometry collision box size=0.7278620044322212 0.38433860865569613 1.1778489928250107; visual box size=0.7278620044322212 0.38433860865569613 1.1778489928250107
- link Link1: mass 0.15136330318765737 -> 0.9404630224771322; geometry collision box size=1.1459699670066485 0.7415451500169353 1.106702496517792; visual box size=1.1459699670066485 0.7415451500169353 1.106702496517792
- link Link2: mass 0.41502688459911957 -> 0.40440714791700105; geometry collision box size=0.6685780257640986 0.9334649001663011 0.6479906394079225; visual box size=0.6685780257640986 0.9334649001663011 0.6479906394079225
- link Link3: mass 1.1863161466101886 -> 0.40360436489446866; geometry collision box size=0.7557420174508104 0.4395517028339273 1.214988924110914; visual box size=0.7557420174508104 0.4395517028339273 1.214988924110914
- link Link4: mass 0.24159438313137246 -> 0.07584981465733509; geometry collision box size=0.5442156882442547 0.35345955611640134 0.3943154002290481; visual box size=0.5442156882442547 0.35345955611640134 0.3943154002290481
- link Link5: mass 0.7124975516153823 -> 0.20777755699414138; geometry collision box size=0.26409229419244296 0.9659456994623945 0.8144983202408741; visual box size=0.26409229419244296 0.9659456994623945 0.8144983202408741
- link Link6: mass 0.23135440586714634 -> 0.8239026012910531; geometry collision box size=1.0445783511847522 0.7570799232841364 1.0418210395041538; visual box size=1.0445783511847522 0.7570799232841364 1.0418210395041538
- link Link7: mass 1.5321151085328013 -> 0.6381685115089957; geometry collision box size=0.9457642142718394 1.0278484768591754 0.6564828689770863; visual box size=0.9457642142718394 1.0278484768591754 0.6564828689770863
- link Link8: mass 0.14599907611527876 -> 0.22064056336946597; geometry collision box size=0.8977706331874812 0.4297942976929744 0.571819963387904; visual box size=0.8977706331874812 0.4297942976929744 0.571819963387904
- link Link9: mass 0.2443504350150486 -> 0.13678303454949609; geometry collision box size=0.4226046201197925 0.6586372250132624 0.4914187479655988; visual box size=0.4226046201197925 0.6586372250132624 0.4914187479655988
Joints:
- joint Link0_Link1: origin xyz=0.333511002351287 0 2 rpy=0 0 0 -> xyz=0.3639310022161106 0 2 rpy=0 0 0
- joint Link1_Link2: axis 1 0 0 -> 0 1 0; origin xyz=0.3429974510710019 -0.13796311591394567 0.0 rpy=0 0 0 -> xyz=0.5729849835033243 0.37077257500846766 0.0 rpy=0 0 0
- joint Link2_Link3: axis 1 0 0 -> 0 1 0; origin xyz=0.0 -0.4790739113090524 0.27045236945647216 rpy=0 0 0 -> xyz=0.3342890128820493 0.46673245008315056 0.0 rpy=0 0 0
- joint Link3_Link4: origin xyz=0.0 0.0 1.2226843599648842 rpy=0 0 0 -> xyz=0.3778710087254052 0.21977585141696365 0.0 rpy=0 0 0
- joint Link4_Link5: origin xyz=0.0 -0.5603661530886882 0.2283595776697132 rpy=0 0 0 -> xyz=0.0 0.35345955611640134 0.0 rpy=0 0 0
- joint Link5_Link6: axis 0 0 1 -> 0 1 0; origin xyz=0.0 -0.2909899026505886 -0.5356145615289158 rpy=0 0 0 -> xyz=0.13204614709622148 0.48297284973119725 0.0 rpy=0 0 0
- joint Link6_Link7: axis 0 1 0 -> 1 0 0; origin xyz=0.0 -0.5149593961200574 -0.34420461572044675 rpy=0 0 0 -> xyz=1.0445783511847522 0.0 0.0 rpy=0 0 0
- joint Link7_Link8: origin xyz=0.0 -0.6092703314104659 0.55959727010696 rpy=0 0 0 -> xyz=0.4728821071359197 -0.5139242384295877 0.0 rpy=0 0 0
- joint Link8_Link9: axis 0 1 0 -> 0 0 1; origin xyz=0.0 0.3759372960743694 0.37288664656707304 rpy=0 0 0 -> xyz=-0.4488853165937406 -0.2148971488464872 0.0 rpy=0 0 0

File: body1.urdf (robot description, URDF)
Before this commit: robot robot, 10 links, 9 joints
Links:
- link Link0: mass 0.16188097376707722 -> 0.09736728915488231; geometry collision box size=0.4007843983721926 0.6193999256119063 0.39222125307278666; visual box size=0.4007843983721926 0.6193999256119063 0.39222125307278666
- link Link1: mass 0.15136330318765737 -> 0.49635385060748777; geometry collision box size=0.9768937533445626 0.7270129944022632 0.6988788367067655; visual box size=0.9768937533445626 0.7270129944022632 0.6988788367067655
- link Link2: mass 0.41502688459911957 -> 0.5822232746195638; geometry collision box size=1.1359979711653514 0.7776187723115614 0.6590908319168599; visual box size=1.1359979711653514 0.7776187723115614 0.6590908319168599
- link Link3: mass 1.1863161466101886 -> 0.11163851655168583; geometry collision box size=0.5188920222126459 0.32201203516976995 0.6681361337253158; visual box size=0.5188920222126459 0.32201203516976995 0.6681361337253158
- link Link4: mass 0.24159438313137246 -> 0.11244251961964398; geometry collision box size=0.2757534824065834 0.541153940552428 0.7535095098483965; visual box size=0.2757534824065834 0.541153940552428 0.7535095098483965
- link Link5: mass 0.7124975516153823 -> 0.40335561970673306; geometry collision box size=1.2159330650197222 0.3593829141935846 0.923041054216622; visual box size=1.2159330650197222 0.3593829141935846 0.923041054216622
- link Link6: mass 0.23135440586714634 -> 0.3031774473683363; geometry collision box size=0.7499323710992 1.0270982292757829 0.3936069978742093; visual box size=0.7499323710992 1.0270982292757829 0.3936069978742093
- link Link7: mass 1.5321151085328013 -> 0.22648028871751005; geometry collision box size=0.33320263643587555 0.6492186053524538 1.0469622519799002; visual box size=0.33320263643587555 0.6492186053524538 1.0469622519799002
- link Link8: mass 0.14599907611527876 -> 0.24287880430138983; geometry collision box size=0.4416757389098901 1.017777192147274 0.5402979970618682; visual box size=0.4416757389098901 1.017777192147274 0.5402979970618682
- link Link9: mass 0.2443504350150486 -> 0.08077572123532749; geometry collision box size=0.46689148761179533 0.26671558907700643 0.6486590599223787; visual box size=0.46689148761179533 0.26671558907700643 0.6486590599223787
Joints:
- joint Link0_Link1: origin xyz=0.333511002351287 0 2 rpy=0 0 0 -> xyz=0.2003921991860963 0 2 rpy=0 0 0
- joint Link1_Link2: origin xyz=0.3429974510710019 -0.13796311591394567 0.0 rpy=0 0 0 -> xyz=0.4884468766722813 0.0 -0.34943941835338277 rpy=0 0 0
- joint Link2_Link3: axis 1 0 0 -> 0 0 1; origin xyz=0.0 -0.4790739113090524 0.27045236945647216 rpy=0 0 0 -> xyz=0.0 0.3888093861557807 -0.32954541595842995 rpy=0 0 0
- joint Link3_Link4: axis 1 0 0 -> 0 0 1; origin xyz=0.0 0.0 1.2226843599648842 rpy=0 0 0 -> xyz=0.0 0.16100601758488498 0.3340680668626579 rpy=0 0 0
- joint Link4_Link5: axis 0 0 1 -> 0 1 0; origin xyz=0.0 -0.5603661530886882 0.2283595776697132 rpy=0 0 0 -> xyz=0.0 0.270576970276214 0.37675475492419824 rpy=0 0 0
- joint Link5_Link6: origin xyz=0.0 -0.2909899026505886 -0.5356145615289158 rpy=0 0 0 -> xyz=0.0 0.3593829141935846 0.0 rpy=0 0 0
- joint Link6_Link7: axis 0 1 0 -> 0 0 1; origin xyz=0.0 -0.5149593961200574 -0.34420461572044675 rpy=0 0 0 -> xyz=0.0 0.5135491146378914 0.19680349893710464 rpy=0 0 0
- joint Link7_Link8: axis 1 0 0 -> 0 0 1; origin xyz=0.0 -0.6092703314104659 0.55959727010696 rpy=0 0 0 -> xyz=-0.16660131821793778 0.0 0.5234811259899501 rpy=0 0 0
- joint Link8_Link9: origin xyz=0.0 0.3759372960743694 0.37288664656707304 rpy=0 0 0 -> xyz=-0.22083786945494505 0.0 -0.2701489985309341 rpy=0 0 0
