Commit message: Finishing up simulations for final project

File: body0.urdf (robot description, URDF)
Before this commit: robot robot, 10 links, 9 joints
Links:
- link Link0: mass 0.32949792017734864 -> 0.2651346497260236; geometry collision box size=0.46196016464367595 1.0486042447602102 0.5473313815072722; visual box size=0.46196016464367595 1.0486042447602102 0.5473313815072722
- link Link1: mass 0.9404630224771322 -> 0.2561138967256754; geometry collision box size=0.27760601195450363 0.843432449464621 1.093840428931189; visual box size=0.27760601195450363 0.843432449464621 1.093840428931189
- link Link2: mass 0.40440714791700105 -> 0.48022449319602734; geometry collision box size=0.6310161240622142 0.9998583107261434 0.7611414782971282; visual box size=0.6310161240622142 0.9998583107261434 0.7611414782971282
- link Link3: mass 0.40360436489446866 -> 1.0082234778663046; geometry collision box size=0.7909518049621886 1.2094343210617524 1.053960891498647; visual box size=0.7909518049621886 1.2094343210617524 1.053960891498647
- link Link4: mass 0.07584981465733509 -> 0.19366326414780405; geometry collision box size=0.282323066623574 0.9593872512312951 0.7150014815635061; visual box size=0.282323066623574 0.9593872512312951 0.7150014815635061
- link Link5: mass 0.20777755699414138 -> 0.2919201297914816; geometry collision box size=1.1975489413951 0.4714327343234883 0.5170720196843658; visual box size=1.1975489413951 0.4714327343234883 0.5170720196843658
- link Link6: mass 0.8239026012910531 -> 0.08075928694853524; geometry collision box size=0.331473964877262 0.6786188286637865 0.3590187640190683; visual box size=0.331473964877262 0.6786188286637865 0.3590187640190683
- link Link7: mass 0.6381685115089957 -> 0.8810877779592906; geometry collision box size=0.8837867606119179 1.0529632373737379 0.9468004961201785; visual box size=0.8837867606119179 1.0529632373737379 0.9468004961201785
- link Link8: mass 0.22064056336946597 -> 0.6597668308845273; geometry collision box size=1.0162113810757705 0.5924541198435198 1.0958514830276775; visual box size=1.0162113810757705 0.5924541198435198 1.0958514830276775
- link Link9: mass 0.13678303454949609 -> 0.6389695247339064; geometry collision box size=0.6787687749994425 1.0740098704123189 0.8764961586242938; visual box size=0.6787687749994425 1.0740098704123189 0.8764961586242938
Joints:
- joint Link0_Link1: origin xyz=0.3639310022161106 0 2 rpy=0 0 0 -> xyz=0.23098008232183798 0 2 rpy=0 0 0
- joint Link1_Link2: axis 0 1 0 -> 1 0 0; origin xyz=0.5729849835033243 0.37077257500846766 0.0 rpy=0 0 0 -> xyz=0.13880300597725181 0.4217162247323105 0.0 rpy=0 0 0
- joint Link2_Link3: axis 0 1 0 -> 0 0 1; origin xyz=0.3342890128820493 0.46673245008315056 0.0 rpy=0 0 0 -> xyz=0.0 0.9998583107261434 0.0 rpy=0 0 0
- joint Link3_Link4: axis 1 0 0 -> 0 0 1; origin xyz=0.3778710087254052 0.21977585141696365 0.0 rpy=0 0 0 -> xyz=0.0 0.6047171605308762 -0.5269804457493235 rpy=0 0 0
- joint Link4_Link5: axis 0 0 1 -> 0 1 0; origin xyz=0.0 0.35345955611640134 0.0 rpy=0 0 0 -> xyz=-0.141161533311787 0.0 -0.35750074078175303 rpy=0 0 0
- joint Link5_Link6: axis 0 1 0 -> 0 0 1; origin xyz=0.13204614709622148 0.48297284973119725 0.0 rpy=0 0 0 -> xyz=-0.59877447069755 0.0 0.2585360098421829 rpy=0 0 0
- joint Link6_Link7: axis 1 0 0 -> 0 1 0; origin xyz=1.0445783511847522 0.0 0.0 rpy=0 0 0 -> xyz=0.0 -0.33930941433189327 0.17950938200953415 rpy=0 0 0
- joint Link7_Link8: axis 1 0 0 -> 0 1 0; origin xyz=0.4728821071359197 -0.5139242384295877 0.0 rpy=0 0 0 -> xyz=-0.4418933803059589 -0.5264816186868689 0.0 rpy=0 0 0
- joint Link8_Link9: axis 0 0 1 -> 1 0 0; origin xyz=-0.4488853165937406 -0.2148971488464872 0.0 rpy=0 0 0 -> xyz=-0.5081056905378852 0.0 0.5479257415138388 rpy=0 0 0

File: body1.urdf (robot description, URDF)
Before this commit: robot robot, 10 links, 9 joints
Links:
- link Link0: mass 0.09736728915488231 -> 0.09451515064035952; geometry collision box size=0.42619625557505525 0.582063574366837 0.3809968448109169; visual box size=0.42619625557505525 0.582063574366837 0.3809968448109169
- link Link1: mass 0.49635385060748777 -> 0.7499080844108429; geometry collision box size=1.059490692126582 0.5947366526832935 1.1901074823333673; visual box size=1.059490692126582 0.5947366526832935 1.1901074823333673
- link Link2: mass 0.5822232746195638 -> 1.028179208492575; geometry collision box size=0.83201417994708 1.128831984411844 1.0947344453922219; visual box size=0.83201417994708 1.128831984411844 1.0947344453922219
- link Link3: mass 0.11163851655168583 -> 0.6531558593400716; geometry collision box size=1.1553923187086492 0.709880265816807 0.7963468160203733; visual box size=1.1553923187086492 0.709880265816807 0.7963468160203733
- link Link4: mass 0.11244251961964398 -> 0.4158423847477743; geometry collision box size=1.0486035911520393 0.5357188517341476 0.7402535226199277; visual box size=1.0486035911520393 0.5357188517341476 0.7402535226199277
- link Link5: mass 0.40335561970673306 -> 0.1901772574919075; geometry collision box size=0.8491103076458784 0.2655332755508357 0.8434814081966372; visual box size=0.8491103076458784 0.2655332755508357 0.8434814081966372
- link Link6: mass 0.3031774473683363 -> 0.40861116435745926; geometry collision box size=0.6836763489894583 1.0573605288848413 0.565244803095373; visual box size=0.6836763489894583 1.0573605288848413 0.565244803095373
- link Link7: mass 0.22648028871751005 -> 0.41063817226717336; geometry collision box size=1.1428887085251513 0.8278572152845355 0.43401020162746506; visual box size=1.1428887085251513 0.8278572152845355 0.43401020162746506
- link Link8: mass 0.24287880430138983 -> 0.2719159404158298; geometry collision box size=1.0379292338255044 0.8620311770449339 0.30390927207375296; visual box size=1.0379292338255044 0.8620311770449339 0.30390927207375296
- link Link9: mass 0.08077572123532749 -> 0.7276369817669347; geometry collision box size=0.6701936800011322 0.9290688365654296 1.1686017779775257; visual box size=0.6701936800011322 0.9290688365654296 1.1686017779775257
Joints:
- joint Link0_Link1: origin xyz=0.2003921991860963 0 2 rpy=0 0 0 -> xyz=0.21309812778752762 0 2 rpy=0 0 0
- joint Link1_Link2: origin xyz=0.4884468766722813 0.0 -0.34943941835338277 rpy=0 0 0 -> xyz=0.529745346063291 0.0 -0.5950537411666836 rpy=0 0 0
- joint Link2_Link3: origin xyz=0.0 0.3888093861557807 -0.32954541595842995 rpy=0 0 0 -> xyz=0.0 0.564415992205922 -0.5473672226961109 rpy=0 0 0
- joint Link3_Link4: origin xyz=0.0 0.16100601758488498 0.3340680668626579 rpy=0 0 0 -> xyz=0.0 0.3549401329084035 0.39817340801018664 rpy=0 0 0
- joint Link4_Link5: origin xyz=0.0 0.270576970276214 0.37675475492419824 rpy=0 0 0 -> xyz=0.0 0.2678594258670738 0.37012676130996386 rpy=0 0 0
- joint Link5_Link6: origin xyz=0.0 0.3593829141935846 0.0 rpy=0 0 0 -> xyz=0.0 0.2655332755508357 0.0 rpy=0 0 0
- joint Link6_Link7: origin xyz=0.0 0.5135491146378914 0.19680349893710464 rpy=0 0 0 -> xyz=0.0 0.5286802644424207 0.2826224015476865 rpy=0 0 0
- joint Link7_Link8: origin xyz=-0.16660131821793778 0.0 0.5234811259899501 rpy=0 0 0 -> xyz=-0.5714443542625757 0.0 0.21700510081373253 rpy=0 0 0
- joint Link8_Link9: origin xyz=-0.22083786945494505 0.0 -0.2701489985309341 rpy=0 0 0 -> xyz=-0.5189646169127522 0.0 -0.15195463603687648 rpy=0 0 0
